Commit message: extended scenario for testes

File: robotino_gazebo_worlds/objects/blue_ball.urdf (robot description, URDF)
Before this commit: robot white_ball, 1 links, 0 joints
Links:
- removed link white_ball
- added link blue_ball, mass 0.01; collision sphere radius=0.10; visual sphere radius=0.10

Commit message: 3 onbj

File: robotino_gazebo_worlds/objects/blue_ball.urdf (robot description, URDF)
Before this commit: robot blue_ball, 1 links, 0 joints
Links:
- link blue_ball: geometry collision sphere radius=0.10; visual sphere radius=0.150

File: robotino_gazebo_worlds/objects/green_cylinder.urdf (robot description, URDF)
Before this commit: robot green_cylinder, 1 links, 0 joints
Links:
- link green_cylinder: geometry collision cylinder length=0.30 radius=0.20; visual cylinder length=0.30 radius=0.20

File: robotino_gazebo_worlds/objects/simple_blue_box2.urdf (robot description, URDF)
Before this commit: robot simple_blue_box2, 1 links, 0 joints
Links:
- link simple_blue_box2: geometry collision box size=0.3 0.3 0.1; visual box size=0.3 0.3 0.1

Commit message: higher objects

File: robotino_gazebo_worlds/objects/blue_ball.urdf (robot description, URDF)
Before this commit: robot blue_ball, 1 links, 0 joints
Links:
- link blue_ball: mass 0.01 -> 2.0; geometry collision cylinder length=0.30 radius=0.15; visual cylinder length=0.30 radius=0.15

File: robotino_gazebo_worlds/objects/simple_blue_box2.urdf (robot description, URDF)
Before this commit: robot simple_blue_box2, 1 links, 0 joints
Links:
- link simple_blue_box2: geometry collision box size=0.3 0.3 0.1; visual box size=0.3 0.3 0.3
